Commit message: Update ur5e_gripper_hand.ros2_control.xacro

File: moveit2_ur5e/config/ur5e_gripper_hand.ros2_control.xacro (robot description, xacro)
@@ -16,4 +16,13 @@
                 <state_interface name="velocity"/>
             </joint>
+            <joint name="robotiq_85_right_knuckle_joint">
+                <param name="mimic">robotiq_85_left_knuckle_joint</param>
+                <param name="multiplier">1</param>
+                <command_interface name="position"/>
+                <state_interface name="position">
+                  <param name="initial_value">0.0</param>
+                </state_interface>
+                <state_interface name="velocity"/>
+            </joint>
         </ros2_control>
     </xacro:macro>

Commit message: Update ur5e_gripper_hand.ros2_control.xacro

File: moveit2_ur5e/config/ur5e_gripper_hand.ros2_control.xacro (robot description, xacro)
@@ -1,5 +1,5 @@
 <?xml version="1.0"?>
 <robot xmlns:xacro="http://www.ros.org/wiki/xacro">
-    <xacro:macro name="ur5e_gripper__hand_ros2_control">
+    <xacro:macro name="ur5e_gripper_hand_ros2_control">
         <ros2_control name="${name}" type="system">
             <hardware>

Commit message: Update ur5e_gripper_hand.ros2_control.xacro

File: moveit2_ur5e/config/ur5e_gripper_hand.ros2_control.xacro (robot description, xacro)
@@ -1,5 +1,5 @@
 <?xml version="1.0"?>
 <robot xmlns:xacro="http://www.ros.org/wiki/xacro">
-    <xacro:macro name="ur5e_gripper_hand_ros2_control">
+    <xacro:macro name="ur5e_gripper_hand_ros2_control" params="name ros2_control_hardware_type">
         <ros2_control name="${name}" type="system">
             <hardware>
