Commit message: Update ur5e_gripper.ros2_control.xacro

File: moveit2_ur5e/config/ur5e_gripper.ros2_control.xacro (robot description, xacro)
@@ -59,4 +59,11 @@
                 <state_interface name="velocity"/>
             </joint>
+            <joint name="robotiq_85_right_knuckle_joint">
+                <command_interface name="position"/>
+                <state_interface name="position">
+                  <param name="initial_value">0.0</param>
+                </state_interface>
+                <state_interface name="velocity"/>
+            </joint>
         </ros2_control>
     </xacro:macro>

Commit message: Update ur5e_gripper.ros2_control.xacro

File: moveit2_ur5e/config/ur5e_gripper.ros2_control.xacro (robot description, xacro)
@@ -59,11 +59,4 @@
                 <state_interface name="velocity"/>
             </joint>
-            <joint name="robotiq_85_right_knuckle_joint">
-                <command_interface name="position"/>
-                <state_interface name="position">
-                  <param name="initial_value">0.0</param>
-                </state_interface>
-                <state_interface name="velocity"/>
-            </joint>
         </ros2_control>
     </xacro:macro>

Commit message: Update ur5e_gripper.ros2_control.xacro

File: moveit2_ur5e/config/ur5e_gripper.ros2_control.xacro (robot description, xacro)
@@ -52,11 +52,4 @@
                 <state_interface name="velocity"/>
             </joint>
-            <joint name="robotiq_85_left_knuckle_joint">
-                <command_interface name="position"/>
-                <state_interface name="position">
-                  <param name="initial_value">${initial_positions['robotiq_85_left_knuckle_joint']}</param>
-                </state_interface>
-                <state_interface name="velocity"/>
-            </joint>
         </ros2_control>
     </xacro:macro>

Commit message: Update ur5e_gripper.ros2_control.xacro

File: moveit2_ur5e/config/ur5e_gripper.ros2_control.xacro (robot description, xacro)
@@ -52,4 +52,20 @@
                 <state_interface name="velocity"/>
             </joint>
+            <joint name="robotiq_85_left_knuckle_joint">
+                <command_interface name="position"/>
+                <state_interface name="position">
+                  <param name="initial_value">${initial_positions['robotiq_85_left_knuckle_joint']}</param>
+                </state_interface>
+                <state_interface name="velocity"/>
+            </joint>
+            <joint name="robotiq_85_right_knuckle_joint">
+                <param name="mimic">robotiq_85_left_knuckle_joint</param>
+                <param name="multiplier">1</param>
+                <command_interface name="position"/>
+                <state_interface name="position">
+                  <param name="initial_value">0.0</param>
+                </state_interface>
+                <state_interface name="velocity"/>
+            </joint>
         </ros2_control>
     </xacro:macro>

Commit message: Update ur5e_gripper.ros2_control.xacro

File: moveit2_ur5e/config/ur5e_gripper.ros2_control.xacro (robot description, xacro)
@@ -68,4 +68,13 @@
                 <state_interface name="velocity"/>
             </joint>
+            <joint name="robotiq_85_left_inner_knuckle_joint">
+                <param name="mimic">robotiq_85_left_knuckle_joint</param>
+                <param name="multiplier">1</param>
+                <command_interface name="position"/>
+                <state_interface name="position">
+                  <param name="initial_value">0.0</param>
+                </state_interface>
+                <state_interface name="velocity"/>
+            </joint>
         </ros2_control>
     </xacro:macro>

Commit message: Update ur5e_gripper.ros2_control.xacro

File: moveit2_ur5e/config/ur5e_gripper.ros2_control.xacro (robot description, xacro)
@@ -77,4 +77,13 @@
                 <state_interface name="velocity"/>
             </joint>
+            <joint name="robotiq_85_right_inner_knuckle_joint">
+                <param name="mimic">robotiq_85_left_knuckle_joint</param>
+                <param name="multiplier">1</param>
+                <command_interface name="position"/>
+                <state_interface name="position">
+                  <param name="initial_value">0.0</param>
+                </state_interface>
+                <state_interface name="velocity"/>
+            </joint>
         </ros2_control>
     </xacro:macro>

Commit message: Update ur5e_gripper.ros2_control.xacro

File: moveit2_ur5e/config/ur5e_gripper.ros2_control.xacro (robot description, xacro)
@@ -86,4 +86,22 @@
                 <state_interface name="velocity"/>
             </joint>
+            <joint name="robotiq_85_left_finger_tip_joint">
+                <param name="mimic">robotiq_85_left_knuckle_joint</param>
+                <param name="multiplier">-1</param>
+                <command_interface name="position"/>
+                <state_interface name="position">
+                  <param name="initial_value">0.0</param>
+                </state_interface>
+                <state_interface name="velocity"/>
+            </joint>
+            <joint name="robotiq_85_right_finger_tip_joint">
+                <param name="mimic">robotiq_85_left_knuckle_joint</param>
+                <param name="multiplier">-1</param>
+                <command_interface name="position"/>
+                <state_interface name="position">
+                  <param name="initial_value">0.0</param>
+                </state_interface>
+                <state_interface name="velocity"/>
+            </joint>
         </ros2_control>
     </xacro:macro>

Commit message: Update ur5e_gripper.ros2_control.xacro

File: moveit2_ur5e/config/ur5e_gripper.ros2_control.xacro (robot description, xacro)
@@ -52,56 +52,4 @@
                 <state_interface name="velocity"/>
             </joint>
-            <joint name="robotiq_85_left_knuckle_joint">
-                <command_interface name="position"/>
-                <state_interface name="position">
-                  <param name="initial_value">${initial_positions['robotiq_85_left_knuckle_joint']}</param>
-                </state_interface>
-                <state_interface name="velocity"/>
-            </joint>
-            <joint name="robotiq_85_right_knuckle_joint">
-                <param name="mimic">robotiq_85_left_knuckle_joint</param>
-                <param name="multiplier">1</param>
-                <command_interface name="position"/>
-                <state_interface name="position">
-                  <param name="initial_value">0.0</param>
-                </state_interface>
-                <state_interface name="velocity"/>
-            </joint>
-            <joint name="robotiq_85_left_inner_knuckle_joint">
-                <param name="mimic">robotiq_85_left_knuckle_joint</param>
-                <param name="multiplier">1</param>
-                <command_interface name="position"/>
-                <state_interface name="position">
-                  <param name="initial_value">0.0</param>
-                </state_interface>
-                <state_interface name="velocity"/>
-            </joint>
-            <joint name="robotiq_85_right_inner_knuckle_joint">
-                <param name="mimic">robotiq_85_left_knuckle_joint</param>
-                <param name="multiplier">1</param>
-                <command_interface name="position"/>
-                <state_interface name="position">
-                  <param name="initial_value">0.0</param>
-                </state_interface>
-                <state_interface name="velocity"/>
-            </joint>
-            <joint name="robotiq_85_left_finger_tip_joint">
-                <param name="mimic">robotiq_85_left_knuckle_joint</param>
-                <param name="multiplier">-1</param>
-                <command_interface name="position"/>
-                <state_interface name="position">
-                  <param name="initial_value">0.0</param>
-                </state_interface>
-                <state_interface name="velocity"/>
-            </joint>
-            <joint name="robotiq_85_right_finger_tip_joint">
-                <param name="mimic">robotiq_85_left_knuckle_joint</param>
-                <param name="multiplier">-1</param>
-                <command_interface name="position"/>
-                <state_interface name="position">
-                  <param name="initial_value">0.0</param>
-                </state_interface>
-                <state_interface name="velocity"/>
-            </joint>
         </ros2_control>
     </xacro:macro>
