Commit message: Update ur5e.urdf

File: ur5e_description/urdf/ur5e.urdf (robot description, URDF)
Before this commit: robot ur5e, 11 links, 10 joints
Links:
- link base_link: geometry collision mesh filename=package://moveit_resources_ur5e_description/meshes/ur5e/col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 scale=1.0 1.0 1.0; visual mesh filename=package://moveit_resources_ur5e_description/meshes/ur5e/vis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
- link forearm_link: geometry collision mesh filename=package://moveit_resources_ur5e_description/meshes/ur5e/col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 scale=1.0 1.0 1.0; visual mesh filename=package://moveit_resources_ur5e_description/meshes/ur5e/vis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
- link shoulder_link: geometry collision mesh filename=package://moveit_resources_ur5e_description/meshes/ur5e/col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 scale=1.0 1.0 1.0; visual mesh filename=package://moveit_resources_ur5e_description/meshes/ur5e/vis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
- link upper_arm_link: geometry collision mesh filename=package://moveit_resources_ur5e_description/meshes/ur5e/col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 scale=1.0 1.0 1.0; visual mesh filename=package://moveit_resources_ur5e_description/meshes/ur5e/vis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
- link wrist_1_link: geometry collision mesh filename=package://moveit_resources_ur5e_description/meshes/ur5e/col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 scale=1.0 1.0 1.0; visual mesh filename=package://moveit_resources_ur5e_description/meshes/ur5e/vis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
- link wrist_2_link: geometry collision mesh filename=package://moveit_resources_ur5e_description/meshes/ur5e/col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 scale=1.0 1.0 1.0; visual mesh filename=package://moveit_resources_ur5e_description/meshes/ur5e/vis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
- link wrist_3_link: geometry collision mesh filename=package://moveit_resources_ur5e_description/meshes/ur5e/col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 scale=1.0 1.0 1.0; visual mesh filename=package://moveit_resources_ur5e_description/meshes/ur5e/vis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
