Commit message: Update ur5e_with_gripper.urdf

File: ur5e_description/urdf/ur5e_with_gripper.urdf (robot description, URDF)
Before this commit: robot ur5e_gripper, 20 links, 19 joints
Links:
- removed link robotiq_85_base_link
- removed link robotiq_85_left_finger_link
- removed link robotiq_85_left_finger_tip_link
- removed link robotiq_85_left_inner_knuckle_link
- removed link robotiq_85_left_knuckle_link
- removed link robotiq_85_right_finger_link
- removed link robotiq_85_right_finger_tip_link
- removed link robotiq_85_right_inner_knuckle_link
- removed link robotiq_85_right_knuckle_link
- added link onrobot_rg2_base_link, mass 0.636951; collision mesh filename=package://moveit_resources_ur5e_description/meshes/ur5e/col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; visual mesh filename=package://moveit_resources_ur5e_description/meshes/ur5e/vis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
Joints:
- removed joint robotiq_85_left_finger_joint
- removed joint robotiq_85_left_finger_tip_joint
- removed joint robotiq_85_left_inner_knuckle_joint
- removed joint robotiq_85_left_knuckle_joint
- removed joint robotiq_85_right_finger_joint
- removed joint robotiq_85_right_finger_tip_joint
- removed joint robotiq_85_right_inner_knuckle_joint
- removed joint robotiq_85_right_knuckle_joint
- joint arm_gripper_joint: child robotiq_85_base_link -> onrobot_rg2_base_link; origin xyz=0.0 0.089 0.0 rpy=0.0 0.0 1.5708 -> xyz=0.0 0.04 0.0 rpy=0.0 0.0 0.0
